File: papilio_cam_board/papilio_cam_board.sch (EAGLE design)
At the start: 20 parts, among them U2 V_REG_317SMD

Commit message: modifying design
Parts:
- added C4: (no value), SparkFun:CAP0805
- added JP3: STAND-OFF, SparkFun:STAND-OFF
- added JP4: (no value), SparkFun:M03PTH
Connections:
- new net N$2: CAMERA_PORT.17, JP4.2
- net 3.3V: now also C4.2
- net GND: now also C4.1, JP4.3; no longer CAMERA_PORT.19
- net RESET_CAM: now also CAMERA_PORT.19, JP4.1; no longer CAMERA_PORT.17
Changed lines of the file:
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@@
 <part name="JP7" library="SparkFun" deviceset="STAND-OFF" device=""/>
 <part name="JP2" library="SparkFun" deviceset="STAND-OFF" device=""/>
+<part name="JP3" library="SparkFun" deviceset="STAND-OFF" device=""/>
+<part name="JP4" library="SparkFun" deviceset="M03" device="PTH"/>
+<part name="GND15" library="supply1" deviceset="GND" device=""/>
+<part name="C4" library="SparkFun" deviceset="CAP" device="0805"/>
+<part name="GND16" library="supply1" deviceset="GND" device=""/>
 </parts>
 <sheets>
@@
 <instance part="R5" gate="G$1" x="175.26" y="78.74" rot="R270"/>
 <instance part="U$4" gate="G$1" x="43.18" y="88.9"/>
-<instance part="P+2" gate="G$1" x="55.88" y="93.98"/>
+<instance part="P+2" gate="G$1" x="66.04" y="93.98"/>
 <instance part="GND10" gate="1" x="30.48" y="83.82"/>
 <instance part="GND13" gate="1" x="30.48" y="96.52" rot="R180"/>
-<instance part="GND14" gate="1" x="63.5" y="96.52" rot="R180"/>
+<instance part="GND14" gate="1" x="73.66" y="93.98" rot="R180"/>
 <instance part="JP7" gate="G$1" x="119.38" y="55.88"/>
 <instance part="JP2" gate="G$1" x="20.32" y="20.32"/>
+<instance part="JP3" gate="G$1" x="0" y="35.56"/>
+<instance part="JP4" gate="G$1" x="81.28" y="33.02" rot="R90"/>
+<instance part="GND15" gate="1" x="71.12" y="40.64" rot="R270"/>
+<instance part="C4" gate="G$1" x="58.42" y="96.52"/>
+<instance part="GND16" gate="1" x="68.58" y="104.14" rot="R90"/>
 </instances>
 <busses>
@@
 </segment>
 <segment>
-<pinref part="CAMERA_PORT" gate="A" pin="19"/>
 <pinref part="CAMERA_PORT" gate="A" pin="20"/>
-<wire x1="88.9" y1="55.88" x2="96.52" y2="55.88" width="0.1524" layer="91"/>
 <pinref part="GND7" gate="1" pin="GND"/>
 <wire x1="96.52" y1="55.88" x2="101.6" y2="55.88" width="0.1524" layer="91"/>
 <wire x1="101.6" y1="55.88" x2="101.6" y2="53.34" width="0.1524" layer="91"/>
-<junction x="96.52" y="55.88"/>
 </segment>
 <segment>
@@
 <pinref part="U$4" gate="G$1" pin="WP"/>
 <pinref part="GND14" gate="1" pin="GND"/>
-<wire x1="55.88" y1="91.44" x2="63.5" y2="91.44" width="0.1524" layer="91"/>
-<wire x1="63.5" y1="91.44" x2="63.5" y2="93.98" width="0.1524" layer="91"/>
+<wire x1="55.88" y1="91.44" x2="73.66" y2="91.44" width="0.1524" layer="91"/>
+</segment>
+<segment>
+<pinref part="JP4" gate="G$1" pin="3"/>
+<pinref part="GND15" gate="1" pin="GND"/>
+<wire x1="73.66" y1="40.64" x2="78.74" y2="40.64" width="0.1524" layer="91"/>
+</segment>
+<segment>
+<pinref part="C4" gate="G$1" pin="1"/>
+<pinref part="GND16" gate="1" pin="GND"/>
+<wire x1="66.04" y1="104.14" x2="58.42" y2="101.6" width="0.1524" layer="91"/>
 </segment>
 </net>
@@
 <pinref part="U$4" gate="G$1" pin="VCC"/>
 <pinref part="P+2" gate="G$1" pin="3.3V"/>
+<wire x1="66.04" y1="93.98" x2="58.42" y2="93.98" width="0.1524" layer="91"/>
+<pinref part="C4" gate="G$1" pin="2"/>
+<wire x1="58.42" y1="93.98" x2="55.88" y2="93.98" width="0.1524" layer="91"/>
+<junction x="58.42" y="93.98"/>
 </segment>
 </net>
@@
 </segment>
 <segment>
-<pinref part="CAMERA_PORT" gate="A" pin="17"/>
-<wire x1="88.9" y1="58.42" x2="78.74" y2="58.42" width="0.1524" layer="91"/>
-<label x="78.74" y="58.42" size="1.778" layer="95"/>
+<pinref part="JP4" gate="G$1" pin="1"/>
+<wire x1="83.82" y1="40.64" x2="101.6" y2="40.64" width="0.1524" layer="91"/>
+<label x="88.9" y="40.64" size="1.778" layer="95"/>
+<pinref part="CAMERA_PORT" gate="A" pin="19"/>
+<wire x1="88.9" y1="55.88" x2="83.82" y2="55.88" width="0.1524" layer="91"/>
+<wire x1="83.82" y1="55.88" x2="83.82" y2="40.64" width="0.1524" layer="91"/>
+<junction x="83.82" y="40.64"/>
 </segment>
 </net>
@@
 </segment>
 </net>
+<net name="N$2" class="0">
+<segment>
+<pinref part="CAMERA_PORT" gate="A" pin="17"/>
+<wire x1="88.9" y1="58.42" x2="81.28" y2="58.42" width="0.1524" layer="91"/>
+<wire x1="81.28" y1="58.42" x2="81.28" y2="40.64" width="0.1524" layer="91"/>
+<pinref part="JP4" gate="G$1" pin="2"/>
+</segment>
+</net>

Commit message: modifying design
Parts:
- renumbered U$1 to H
Connections:
- new net N$3: C3.2, R3.1, S1.4
- new net N$4: C3.1, S1.2
- net 3.3V: now also HA_B_POWER.3V3@P14, HA_B_POWER.3V3@P6
- net GND: no longer C3.1, S1.2
- net RESET: no longer C3.2, R3.1, S1.4
Other:
- moved on the sheet: C3, R3, S1

Commit message: reversing some changes
Parts:
- renumbered H to U$1
Connections:
- removed net N$3: C3.2, R3.1, S1.4
- removed net N$4: C3.1, S1.2
- net GND: now also C3.1, S1.2
- net RESET: now also C3.2, R3.1, S1.4
Other:
- moved on the sheet: C3, R3, S1

Commit message: refactoring
Parts:
- added JP6: (no value), SparkFun:M03PTH
Connections:
- new net ALIM_LCD: JP6.2, LCD_INTERFACE.1
- new net LCD_5V: JP6.1, U$1A_B_POWER.5V0@P4
- net 3.3V: now also JP6.3; no longer LCD_INTERFACE.1
- net GND: now also C1.2
- net N$1: no longer C1.2
Changed lines of the file:
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@@
 <part name="LCD_INTERFACE" library="pinhead" deviceset="PINHD-2X12" device=""/>
 <part name="GND12" library="supply1" deviceset="GND" device=""/>
-<part name="P+10" library="SparkFun" deviceset="3.3V" device=""/>
 <part name="LOGO1" library="Papilio" deviceset="BUTTERFLY_LOGO" device=""/>
 <part name="GND7" library="supply1" deviceset="GND" device=""/>
@@
 <part name="P+3" library="SparkFun" deviceset="3.3V" device=""/>
 <part name="P+4" library="SparkFun" deviceset="3.3V" device=""/>
+<part name="JP6" library="SparkFun" deviceset="M03" device="PTH"/>
+<part name="P+7" library="SparkFun" deviceset="3.3V" device=""/>
 </parts>
 <sheets>
@@
 <instance part="LCD_INTERFACE" gate="A" x="-20.32" y="78.74"/>
 <instance part="GND12" gate="1" x="-5.08" y="91.44" rot="R90"/>
-<instance part="P+10" gate="G$1" x="-38.1" y="91.44"/>
 <instance part="LOGO1" gate="G$1" x="142.24" y="60.96"/>
 <instance part="GND7" gate="1" x="101.6" y="50.8"/>
@@
 <instance part="P+3" gate="G$1" x="121.92" y="-25.4" rot="R270"/>
 <instance part="P+4" gate="G$1" x="121.92" y="-5.08" rot="R270"/>
+<instance part="JP6" gate="G$1" x="-66.04" y="78.74" rot="R90"/>
+<instance part="P+7" gate="G$1" x="-68.58" y="96.52"/>
 </instances>
 <busses>
@@
 <wire x1="25.4" y1="-25.4" x2="12.7" y2="-25.4" width="0.1524" layer="91"/>
 <junction x="12.7" y="-25.4"/>
+<pinref part="C1" gate="G$1" pin="2"/>
+<wire x1="0" y1="-12.7" x2="0" y2="-25.4" width="0.1524" layer="91"/>
+<wire x1="0" y1="-25.4" x2="12.7" y2="-25.4" width="0.1524" layer="91"/>
 </segment>
 <segment>
@@
 </segment>
 <segment>
-<pinref part="P+10" gate="G$1" pin="3.3V"/>
-<pinref part="LCD_INTERFACE" gate="A" pin="1"/>
-<wire x1="-38.1" y1="91.44" x2="-22.86" y2="91.44" width="0.1524" layer="91"/>
-</segment>
-<segment>
 <pinref part="FIFO_INTERFACE" gate="A" pin="16"/>
 <pinref part="P+9" gate="G$1" pin="3.3V"/>
@@
 <pinref part="P+4" gate="G$1" pin="3.3V"/>
 </segment>
+<segment>
+<pinref part="P+7" gate="G$1" pin="3.3V"/>
+<pinref part="JP6" gate="G$1" pin="3"/>
+<wire x1="-68.58" y1="96.52" x2="-68.58" y2="86.36" width="0.1524" layer="91"/>
+</segment>
 </net>
 <net name="N$1" class="0">
@@
 <wire x1="20.32" y1="-15.24" x2="12.7" y2="-15.24" width="0.1524" layer="91"/>
 <junction x="12.7" y="-15.24"/>
-<pinref part="C1" gate="G$1" pin="2"/>
-<wire x1="12.7" y1="-15.24" x2="0" y2="-15.24" width="0.1524" layer="91"/>
-<wire x1="0" y1="-15.24" x2="0" y2="-12.7" width="0.1524" layer="91"/>
 </segment>
 </net>
@@
 </segment>
 </net>
+<net name="ALIM_LCD" class="0">
+<segment>
+<pinref part="JP6" gate="G$1" pin="2"/>
+<wire x1="-66.04" y1="86.36" x2="-66.04" y2="104.14" width="0.1524" layer="91"/>
+<wire x1="-66.04" y1="104.14" x2="-38.1" y2="104.14" width="0.1524" layer="91"/>
+<label x="-43.18" y="104.14" size="1.778" layer="95"/>
+<pinref part="LCD_INTERFACE" gate="A" pin="1"/>
+<wire x1="-38.1" y1="91.44" x2="-22.86" y2="91.44" width="0.1524" layer="91"/>
+<wire x1="-38.1" y1="104.14" x2="-38.1" y2="91.44" width="0.1524" layer="91"/>
+</segment>
+</net>
+<net name="LCD_5V" class="0">
+<segment>
+<pinref part="U$1" gate="A_B_POWER" pin="5V0@P4"/>
+<wire x1="96.52" y1="0" x2="83.82" y2="0" width="0.1524" layer="91"/>
+<label x="83.82" y="0" size="1.778" layer="95"/>
+</segment>
+<segment>
+<pinref part="JP6" gate="G$1" pin="1"/>
+<wire x1="-63.5" y1="96.52" x2="-63.5" y2="86.36" width="0.1524" layer="91"/>
+<wire x1="-63.5" y1="96.52" x2="-50.8" y2="96.52" width="0.1524" layer="91"/>
+<label x="-58.42" y="96.52" size="1.778" layer="95"/>
+</segment>
+</net>
